File: flex/flex.kicad_pcb (KiCad board)
At the start: 2 copper layers, 48.8 x 41.5 mm, 10 parts, among them J1 Conn_01x06_Female, J2 Conn_01x03_Female, SW19 SW_Push, SW5 SW_Push, SW9 SW_Push

Commit message: have I broken the holes again?
Parts:
- added D10: SK6812MINI, libs2:YS-SK6812MINI-E_REVERSE, F.Cu at (94.2, 79.2)
- added D11: SK6812MINI, libs2:YS-SK6812MINI-E_REVERSE_NO_EDGECUT, B.Cu at (94.2, 79.2)
- added D12: SK6812MINI, libs2:YS-SK6812MINI-E_REVERSE, F.Cu at (74.8, 80.8)
- added D13: SK6812MINI, libs2:YS-SK6812MINI-E_REVERSE_NO_EDGECUT, B.Cu at (74.8, 80.8)
- added D2: SK6812MINI, libs2:YS-SK6812MINI-E_REVERSE, F.Cu at (76.5, 102.8)
- added D3: SK6812MINI, libs2:YS-SK6812MINI-E_REVERSE_NO_EDGECUT, B.Cu at (76.5, 102.8)
- added R1: R, Resistor_SMD:R_1206_3216Metric_Pad1.42x1.75mm_HandSolder, B.Cu at (81.1, 79.1)
- added R2: R, Resistor_SMD:R_1206_3216Metric_Pad1.42x1.75mm_HandSolder, F.Cu at (81.2, 79.2)
Connections:
- D19 pad 2: Net-(D19-A) -> (no net)
- D5 pad 2: Net-(D5-A) -> (no net)
- D9 pad 2: Net-(D9-A) -> (no net)
- J1 pad 1: unconnected-(J1-Pin_1-Pad1) -> (no net)
- J1 pad 6: unconnected-(J1-Pin_6-Pad6) -> (no net)
- J2 pad 1: unconnected-(J2-Pin_1-Pad1) -> (no net)
Routing:
- net Vcc: track 0.00 -> 74.8 mm, vias 0 -> 4
- net Net-(D10-Pad1): track 0.00 -> 69.9 mm, vias 0 -> 3
- net Gnd: track 0.00 -> 57.6 mm, vias 0 -> 2
- net Net-(D12-Pad1): track 0.00 -> 27.2 mm, vias 0 -> 3
- net Net-(D12-Pad3): track 0.00 -> 19.5 mm, vias 0 -> 3
- net col6: track 78.6 -> 59.3 mm, vias 4 -> 3
- net row1: track 62.5 -> 57.8 mm
- net Din: track 0.00 -> 1.95 mm, vias 0 -> 1
Other:
- board text added: "Vcc"
- board text removed: "C"
- board text removed: "Row"

Commit message: cleaned
Parts:
- removed D10, D12, D2: SK6812MINI, libs2:YS-SK6812MINI-E_REVERSE
- removed D11, D13, D3: SK6812MINI, libs2:YS-SK6812MINI-E_REVERSE_NO_EDGECUT
- removed R1, R2: R, Resistor_SMD:R_1206_3216Metric_Pad1.42x1.75mm_HandSolder
Connections:
- D19 pad 2: (no net) -> Net-(D19-Pad2)
- D5 pad 2: (no net) -> Net-(D5-Pad2)
- D9 pad 2: (no net) -> Net-(D9-Pad2)
- J1 pad 1: (no net) -> unconnected-(J1-Pad1)
- J1 pad 6: (no net) -> unconnected-(J1-Pad6)
- J2 pad 1: (no net) -> Vcc
- J2 pad 2: row1 -> Gnd
- J2 pad 3: col6 -> Din
- SW19 pad 2: Net-(D19-A) -> Net-(D19-Pad2)
- SW5 pad 2: Net-(D5-A) -> Net-(D5-Pad2)
- SW9 pad 2: Net-(D9-A) -> Net-(D9-Pad2)
Routing:
- net Vcc: track 74.8 -> 0.00 mm, vias 4 -> 0
- net Net-(D10-Pad1): track 69.9 -> 0.00 mm, vias 3 -> 0
- net Gnd: track 57.6 -> 0.42 mm, vias 2 -> 0
- net Net-(D12-Pad1): track 27.2 -> 0.00 mm, vias 3 -> 0
- net Net-(D12-Pad3): track 19.5 -> 0.00 mm, vias 3 -> 0
- net Net-(D19-Pad2): track 0.00 -> 11.7 mm, vias 0 -> 1
- net Net-(D19-A): track 11.7 -> 0.00 mm, vias 1 -> 0
- net Net-(D9-Pad2): track 0.00 -> 8.50 mm, vias 0 -> 1
- net Net-(D9-A): track 8.50 -> 0.00 mm, vias 1 -> 0
- net Net-(D5-Pad2): track 0.00 -> 6.63 mm
- net Net-(D5-A): track 6.63 -> 0.00 mm
- net col6: track 59.3 -> 54.0 mm
- net Din: track 1.95 -> 0.00 mm, vias 1 -> 0
- added copper zone on B.Cu, net Gnd
- added copper zone on F.Cu, net Gnd
- removed copper zone on B.Cu, net row1
- removed copper zone on F.Cu, net row1
Other:
- board text removed: "R"

Commit message: routed
Connections:
- J2 pad 1: Vcc -> unconnected-(J2-Pin_1-Pad1)
- J2 pad 2: Gnd -> row1
- J2 pad 3: Din -> col6
Routing:
- net col6: track 54.0 -> 58.2 mm
- added copper zone on B.Cu, net row1
- added copper zone on F.Cu, net row1
- removed copper zone on B.Cu, net Gnd
- removed copper zone on F.Cu, net Gnd
Other:
- board text added: "C"
- board text added: "R"
- board text added: "REV O"
- board text removed: "Vcc"
